File: pcb/pumpenonkel.kicad_pcb (KiCad board)
At the start: 2 copper layers, 121.4 x 144.2 mm, 55 parts, among them J1 Conn_01x03_Pin, J10 CHANNEL, J11 CHANNEL, J12 CHANNEL, J13 Screw_Terminal_01x02, J14 Screw_Terminal_01x02, J15 CHANNEL, J16 Conn_01x03_Pin, J17 Barrel_Jack, J2 Conn_01x03_Pin, J3 Conn_01x03_Pin, J4 Conn_01x03_Pin, J5 Conn_01x03_Pin, J6 Conn_01x03_Pin, J7 Conn_01x08_Pin, J8 CHANNEL, J9 CHANNEL, K1 SANYOU_SRD_Form_C, K2 SANYOU_SRD_Form_C, K3 SANYOU_SRD_Form_C, K4 SANYOU_SRD_Form_C, K5 SANYOU_SRD_Form_C, K6 SANYOU_SRD_Form_C, Q1 BC337, Q2 BC337, Q3 BC337, Q4 BC337, Q5 BC337, Q6 BC337

Commit message: Fix some bugs
Connections:
- A1 pad 39: Net-(A1-VSYS) -> VCC_BRIDGE
- J16 pad 3: Net-(A1-VSYS) -> VCC_BRIDGE
- J7 pad 1: VCC -> VCC_BRIDGE
Routing:
- net VCC_BRIDGE: track 0.00 -> 79.3 mm
- net VCC: track 392.5 -> 322.0 mm
- net Net-(A1-VSYS): track 12.6 -> 0.00 mm
