File: pcb/pumpenonkel.kicad_sch (KiCad schematic)
At the start: 7 parts, among them J13 Screw_Terminal_01x02, J14 Screw_Terminal_01x02, J16 Conn_01x03_Pin, J17 Barrel_Jack, J7 Conn_01x08_Pin

Commit message: Fix some bugs
Connections:
- net VCC: no longer J7.1 (Pin_1)
- net VCC_BRIDGE: now reaches A1.39 (VSYS), J16.3 (Pin_3)
- net VCC_BRIDGE: now also J7.1 (Pin_1)
