File: pcb/relais_channel.kicad_sch (KiCad schematic)
At the start: 8 parts, among them J3 Conn_01x03_Pin, J8 CHANNEL, K1 SANYOU_SRD_Form_C, Q1 BC337

Commit message: finalilise pcb
Parts:
- Q1: footprint Package_TO_SOT_THT:TO-92_Inline -> Package_TO_SOT_THT:TO-92
Changed lines of the file:
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@@
 			)
 		)
-		(property "Footprint" "Package_TO_SOT_THT:TO-92_Inline"
+		(property "Footprint" "Package_TO_SOT_THT:TO-92"
 			(at 72.39 65.405 0)
 			(effects
